File: control_board/control_board.brd (EAGLE design)
At the start: 107.8 x 40 mm, 86 parts

Commit message: more
Parts:
- added C1, C2: (no value), rcl:C0805
- added IC1: TL072D, linear:SO08
- added R1, R10, R11, R2, R3, R4, R5, R6, R7, R8, R9: (no value), rcl:R0805
- turned +12V to 0 degrees
- turned -12V to 0 degrees
- renumbered AGND1 to -12V, AGND2 to +12V
Connections:
- removed net N$25: +5V.1, LED_VCA1.A, LED_VCA2.A, LED_VCA3.A, LED_VCA4.A
- new net +12V: +12V.1, C1.1, IC1.8
- new net +5V: +5V.1, LED_VCA1.A, LED_VCA2.A, LED_VCA3.A, LED_VCA4.A, R1.1, R2.1, R3.1, R4.1
- new net -12V: -12V.1, C2.1, IC1.4
- new net N$29: CV1.P$2, R1.2
- new net N$30: CV2.P$2, R2.2
- new net N$31: CV3.P$2, R3.2
- new net N$32: CV4.P$2, R4.2
- new net N$34: IN2.P$2, R5.1
- new net N$35: IN3.P$2, R6.1
- new net N$36: IN4.P$2, R7.1
- new net N$37: IN1.P$1, R5.2, SIG_IN1.1
- new net N$38: OUT3.P$2, R10.1
- new net N$39: OUT2.P$2, R9.1
- new net N$42: IC1.3, R10.2, R11.2, R8.2, R9.2
- new net N$44: IC1.1, IC1.2, OUT4.P$1
- new net N$46: IC1.6, IC1.7
- net AGND: now also C1.2, C2.2, IC1.5; no longer +12V.1, -12V.1, IN1.P$2
- net GND: no longer CV1.P$2, CV2.P$2, CV3.P$2, CV4.P$2
- net N$10: now also R6.2; no longer IN3.P$2
- net N$11: now also R7.2; no longer IN4.P$2
- net N$28: now also R11.1; no longer OUT4.P$1
- net N$9: now also OUT1.P$2, R8.1; no longer IN1.P$1, IN2.P$2, SIG_IN1.1
Routing:
- net +5V: track 0.00 -> 124.3 mm
- net N$25: track 99.5 -> 0.00 mm
- net N$42: track 0.00 -> 50.6 mm
- net N$9: track 52.7 -> 2.51 mm
- net N$37: track 0.00 -> 40.7 mm
- net N$44: track 0.00 -> 40.7 mm, vias 0 -> 1
- net +12V: track 0.00 -> 33.2 mm, vias 0 -> 1
- net -12V: track 0.00 -> 32.1 mm
- net N$10: track 62.8 -> 39.7 mm
- net N$11: track 44.6 -> 27.9 mm, vias 0 -> 1
- net SW_READ: track 46.0 -> 58.7 mm
- net N$36: track 0.00 -> 12.4 mm, vias 0 -> 1
- net N$35: track 0.00 -> 12.0 mm, vias 0 -> 1
- net N$34: track 0.00 -> 11.9 mm, vias 0 -> 1
- net SINK4: track 82.7 -> 89.0 mm
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Other:
- board text added: "CONTROL BOARD V1"
- board text added: "DIGITALLY CONTROLLED QUAD VCA/MIXER"
- board text added: "hotchk155"

Commit message: fixes
Parts:
- removed CK_IN, CK_OUT: WQP-PJ301M-12_JACK, thonkiconn:WQP-PJ301M-12_JACK
- removed MIDI: VERTICAL_3_5MM_SOCKET, jason_eagle6:VERTICAL_3_5MM_SOCKET
- removed R1, R2, R3, R4: (no value), rcl:R0805
- added X1: VERTICAL_3_5MM_SOCKETTHONK, jason_eagle6:PJ301CM
- moved LED9 20.1 mm to (41.9, 40.0), turned to 180 degrees
- moved LED10 19.3 mm to (47.0, 40.0), turned to 180 degrees
- moved LED_TRIG1 14.0 mm to (52.1, 56.5)
- moved LED_TRIG2 14.0 mm to (52.1, 66.0)
- moved LED_TRIG3 14.0 mm to (52.1, 37.5)
- moved LED_TRIG4 14.0 mm to (52.1, 47.0)
- moved LED_VCA1 14.0 mm to (52.1, 42.5)
- moved LED_VCA2 14.0 mm to (52.1, 52.1)
- moved LED_VCA3 14.0 mm to (52.1, 61.6)
- moved LED_VCA4 14.0 mm to (52.1, 71.1)
- moved CV1 1.52 mm to (59.8, 40.0), turned to 270 degrees
- moved CV2 1.52 mm to (59.8, 49.5), turned to 270 degrees
- moved CV3 1.52 mm to (59.8, 59.1), turned to 270 degrees
- moved CV4 1.52 mm to (59.8, 68.6), turned to 270 degrees
- turned DGND3 to 0 degrees
- renumbered CKIN to DGND3
Connections:
- removed net N$17: CK_IN.P$1, CK_OUT.P$1, DGND3.1
- removed net N$29: CV1.P$2, R1.2
- removed net N$30: CV2.P$2, R2.2
- removed net N$31: CV3.P$2, R3.2
- removed net N$32: CV4.P$2, R4.2
- net +5V: no longer R1.1, R2.1, R3.1, R4.1
- net GND: now also CV1.P$2, CV2.P$2, CV3.P$2, CV4.P$2, DGND3.1; no longer CK_IN.P$2, CK_IN.P$3, CK_OUT.P$3
- net N$19: now also X1.R; no longer MIDI.3
- net N$20: now also X1.T; no longer MIDI.4
Routing:
- net +5V: track 124.3 -> 65.7 mm, vias 0 -> 1
- net N$17: track 37.3 -> 0.00 mm
- net SINK3: track 112.1 -> 80.6 mm
- net N$22: track 65.3 -> 42.2 mm
- net SINK1: track 92.3 -> 73.5 mm
- net N$24: track 77.9 -> 60.5 mm
- net SINK2: track 72.5 -> 57.4 mm
- net N$23: track 67.4 -> 52.7 mm
- net N$21: track 44.7 -> 30.1 mm, vias 1 -> 0
- net SINK5: track 62.9 -> 48.9 mm
- net N$15: track 52.9 -> 65.1 mm
- net N$13: track 30.2 -> 41.7 mm
- net SINK4: track 89.0 -> 77.7 mm, vias 1 -> 0
- net N$16: track 71.6 -> 81.7 mm, vias 0 -> 2
- net N$19: track 22.5 -> 13.5 mm
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Other:
- board text added: "CONTROL BOARD V2"
