File: control_board/control_board.sch (EAGLE design)
At the start: 86 parts, among them X1 VERTICAL_3_5MM_SOCKET

Commit message: in work
Parts:
- removed SW1, SW2, SW3, SW4, SW_TRG1, SW_TRG2, SW_TRG3, SW_TRG4: (no value), switch-omron:10-XX
- added U$1, U$2, U$3, U$4, U$6, U$7, U$8, U$9: 6MM_TACT, jason_eagle6:6MM_TACT
Connections:
- net GND: now also U$9.1, U$9.4; no longer SW4.P, SW4.P1
- net N$18: no longer OUT1.3
- net N$26: no longer OUT3.3
- net N$27: no longer OUT2.3
- net N$28: no longer OUT4.3
- net SINK1: now also U$1.2, U$1.3; no longer SW_TRG1.S, SW_TRG1.S1
- net SINK2: now also U$2.2, U$2.3; no longer SW_TRG2.S, SW_TRG2.S1
- net SINK3: now also U$3.2, U$3.3; no longer SW_TRG3.S, SW_TRG3.S1
- net SINK4: now also U$4.2, U$4.3; no longer SW_TRG4.S, SW_TRG4.S1
- net SINK5: now also U$6.2, U$6.3; no longer SW1.S, SW1.S1
- net SINK6: now also U$7.2, U$7.3; no longer SW2.S, SW2.S1
- net SINK7: now also U$8.2, U$8.3; no longer SW3.S, SW3.S1
- net SWITCH: now also U$9.2, U$9.3; no longer SW4.S, SW4.S1
- net SW_READ: now also U$1.1, U$1.4, U$2.1, U$2.4, U$3.1, U$3.4, U$4.1, U$4.4, U$6.1, U$6.4, U$7.1, U$7.4, U$8.1, U$8.4; no longer SW1.P, SW1.P1, SW2.P, SW2.P1, SW3.P, SW3.P1, SW_TRG1.P, SW_TRG1.P1, SW_TRG2.P, SW_TRG2.P1, SW_TRG3.P, SW_TRG3.P1, SW_TRG4.P, SW_TRG4.P1

Commit message: moar stuffs
Connections:
- net GND: now also CK_IN.3, CV1.3, CV2.3, CV3.3, CV4.3
Changed lines of the file:
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@@
 <net name="GND" class="0">
 <segment>
-<wire x1="20.32" y1="93.98" x2="33.02" y2="93.98" width="0.1524" layer="91"/>
+<wire x1="20.32" y1="93.98" x2="30.48" y2="93.98" width="0.1524" layer="91"/>
 <pinref part="GND1" gate="1" pin="GND"/>
-<wire x1="33.02" y1="93.98" x2="43.18" y2="93.98" width="0.1524" layer="91"/>
-<wire x1="43.18" y1="93.98" x2="53.34" y2="93.98" width="0.1524" layer="91"/>
-<wire x1="53.34" y1="93.98" x2="63.5" y2="93.98" width="0.1524" layer="91"/>
+<wire x1="30.48" y1="93.98" x2="33.02" y2="93.98" width="0.1524" layer="91"/>
+<wire x1="33.02" y1="93.98" x2="40.64" y2="93.98" width="0.1524" layer="91"/>
+<wire x1="40.64" y1="93.98" x2="43.18" y2="93.98" width="0.1524" layer="91"/>
+<wire x1="43.18" y1="93.98" x2="50.8" y2="93.98" width="0.1524" layer="91"/>
+<wire x1="50.8" y1="93.98" x2="53.34" y2="93.98" width="0.1524" layer="91"/>
+<wire x1="53.34" y1="93.98" x2="60.96" y2="93.98" width="0.1524" layer="91"/>
+<wire x1="60.96" y1="93.98" x2="63.5" y2="93.98" width="0.1524" layer="91"/>
 <wire x1="20.32" y1="93.98" x2="20.32" y2="91.44" width="0.1524" layer="91"/>
 <pinref part="CV4" gate="G$1" pin="1"/>
@@
 <wire x1="33.02" y1="99.06" x2="33.02" y2="93.98" width="0.1524" layer="91"/>
 <junction x="33.02" y="93.98"/>
+<pinref part="CV1" gate="G$1" pin="3"/>
+<wire x1="30.48" y1="99.06" x2="30.48" y2="93.98" width="0.1524" layer="91"/>
+<junction x="30.48" y="93.98"/>
+<pinref part="CV2" gate="G$1" pin="3"/>
+<wire x1="40.64" y1="99.06" x2="40.64" y2="93.98" width="0.1524" layer="91"/>
+<junction x="40.64" y="93.98"/>
+<pinref part="CV3" gate="G$1" pin="3"/>
+<wire x1="50.8" y1="99.06" x2="50.8" y2="93.98" width="0.1524" layer="91"/>
+<junction x="50.8" y="93.98"/>
+<pinref part="CV4" gate="G$1" pin="3"/>
+<wire x1="60.96" y1="99.06" x2="60.96" y2="93.98" width="0.1524" layer="91"/>
+<junction x="60.96" y="93.98"/>
 </segment>
 <segment>
@@
 <pinref part="CK_IN" gate="G$1" pin="1"/>
 <wire x1="30.48" y1="50.8" x2="30.48" y2="53.34" width="0.1524" layer="91"/>
+<pinref part="CK_IN" gate="G$1" pin="3"/>
+<wire x1="30.48" y1="50.8" x2="27.94" y2="50.8" width="0.1524" layer="91"/>
+<wire x1="27.94" y1="50.8" x2="27.94" y2="53.34" width="0.1524" layer="91"/>
+<junction x="30.48" y="50.8"/>
 </segment>
 <segment>

Commit message: and more
Connections:
- net AGND: now also IN1.3
Changed lines of the file:
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@@
 <pinref part="IN2" gate="G$1" pin="1"/>
 <wire x1="45.72" y1="-17.78" x2="45.72" y2="-5.08" width="0.1524" layer="91"/>
+<junction x="45.72" y="-17.78"/>
+<junction x="45.72" y="-5.08"/>
 </segment>
 <segment>
@@
 <pinref part="IN3" gate="G$1" pin="1"/>
 <wire x1="66.04" y1="-17.78" x2="66.04" y2="-5.08" width="0.1524" layer="91"/>
+<junction x="66.04" y="-17.78"/>
+<junction x="66.04" y="-5.08"/>
 </segment>
 <segment>
@@
 <pinref part="IN4" gate="G$1" pin="1"/>
 <wire x1="83.82" y1="-17.78" x2="83.82" y2="-5.08" width="0.1524" layer="91"/>
+<junction x="83.82" y="-17.78"/>
+<junction x="83.82" y="-5.08"/>
 </segment>
 <segment>
@@
 <pinref part="IN1" gate="G$1" pin="1"/>
 <pinref part="SUPPLY5" gate="G$1" pin="AGND"/>
-<wire x1="25.4" y1="-5.08" x2="25.4" y2="-17.78" width="0.1524" layer="91"/>
+<wire x1="25.4" y1="-5.08" x2="25.4" y2="-10.16" width="0.1524" layer="91"/>
+<junction x="25.4" y="-17.78"/>
+<junction x="25.4" y="-5.08"/>
+<pinref part="IN1" gate="G$1" pin="3"/>
+<wire x1="25.4" y1="-10.16" x2="25.4" y2="-17.78" width="0.1524" layer="91"/>
+<wire x1="22.86" y1="-5.08" x2="22.86" y2="-10.16" width="0.1524" layer="91"/>
+<wire x1="22.86" y1="-10.16" x2="25.4" y2="-10.16" width="0.1524" layer="91"/>
+<junction x="25.4" y="-10.16"/>
 </segment>
 <segment>
@@
 <wire x1="43.18" y1="-7.62" x2="43.18" y2="-5.08" width="0.1524" layer="91"/>
 <junction x="20.32" y="-7.62"/>
+<junction x="20.32" y="-17.78"/>
+<junction x="43.18" y="-5.08"/>
+<junction x="20.32" y="-5.08"/>
 </segment>
 </net>
@@
 <wire x1="63.5" y1="-10.16" x2="63.5" y2="-5.08" width="0.1524" layer="91"/>
 <junction x="40.64" y="-10.16"/>
+<junction x="40.64" y="-17.78"/>
+<junction x="63.5" y="-5.08"/>
+<junction x="40.64" y="-5.08"/>
 </segment>
 </net>
@@
 <wire x1="81.28" y1="-7.62" x2="81.28" y2="-5.08" width="0.1524" layer="91"/>
 <junction x="60.96" y="-7.62"/>
+<junction x="60.96" y="-17.78"/>
+<junction x="81.28" y="-5.08"/>
+<junction x="60.96" y="-5.08"/>
 </segment>
 </net>
@@
 <pinref part="IN4" gate="G$1" pin="2"/>
 <wire x1="78.74" y1="-17.78" x2="78.74" y2="-5.08" width="0.1524" layer="91"/>
+<junction x="78.74" y="-17.78"/>
+<junction x="78.74" y="-5.08"/>
 </segment>
 </net>

Commit message: MORE
Parts:
- renumbered U$1 to S2, U$2 to S3, U$3 to S8, U$4 to S4, U$5 to DISP1, U$6 to S5, U$7 to S6, U$8 to S7, U$9 to S1, X1 to MIDI

Commit message: more
Parts:
- removed AGND1, AGND2: (no value), pinhead:PINHD-1X1
- added +12V, -12V: (no value), pinhead:PINHD-1X1
- added C1, C2: (no value), rcl:C-EUC0805
- added IC1: TL072D, linear:TL072D
- added R1, R10, R11, R2, R3, R4, R5, R6, R7, R8, R9: (no value), rcl:R-EU_R0805
Connections:
- removed net N$25: +5V.1, LED_VCA1.A, LED_VCA2.A, LED_VCA3.A, LED_VCA4.A
- new net +12V: +12V.1, C1.1, IC1P.V+
- new net +5V: +5V.1, LED_VCA1.A, LED_VCA2.A, LED_VCA3.A, LED_VCA4.A, R1.1, R2.1, R3.1, R4.1
- new net -12V: -12V.1, C2.1, IC1P.V-
- new net N$29: CV1.3, R1.2
- new net N$30: CV2.3, R2.2
- new net N$31: CV3.3, R3.2
- new net N$32: CV4.3, R4.2
- new net N$34: IN2.3, R5.1
- new net N$35: IN3.3, R6.1
- new net N$36: IN4.3, R7.1
- new net N$37: IN1.2, R5.2, SIG_IN1.1
- new net N$38: OUT3.3, R10.1
- new net N$39: OUT2.3, R9.1
- new net N$42: IC1A.+IN, R10.2, R11.2, R8.2, R9.2
- new net N$44: IC1A.-IN, IC1A.OUT, OUT4.2
- new net N$46: IC1B.-IN, IC1B.OUT
- net AGND: now also C1.2, C2.2, IC1B.+IN; no longer AGND1.1, AGND2.1, IN1.3
- net GND: no longer CV1.3, CV2.3, CV3.3, CV4.3
- net N$10: now also R6.2; no longer IN3.3
- net N$11: now also R7.2; no longer IN4.3
- net N$28: now also R11.1; no longer OUT4.2
- net N$9: now also OUT1.3, R8.1; no longer IN1.2, IN2.3, SIG_IN1.1
Other:
- moved on the sheet: ATT1, ATT2, ATT3, ATT4, ATT_IN1, ATT_IN2, ATT_IN3, ATT_IN4, ATT_OUT1, ATT_OUT2, ATT_OUT3, ATT_OUT4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

Commit message: fixes
Parts:
- removed CKIN: (no value), pinhead:PINHD-1X1
- removed CK_IN, CK_OUT: WQP-PJ301M-12_JACK, thonkiconn:WQP-PJ301M-12_JACK
- removed MIDI: VERTICAL_3_5MM_SOCKET, jason_eagle6:VERTICAL_3_5MM_SOCKET
- removed R1, R2, R3, R4: (no value), rcl:R-EU_R0805
- added DGND3: (no value), pinhead:PINHD-1X1
- added X1: VERTICAL_3_5MM_SOCKETTHONK, jason_eagle6:VERTICAL_3_5MM_SOCKETTHONK
Connections:
- removed net N$17: CKIN.1, CK_IN.2, CK_OUT.2
- removed net N$29: CV1.3, R1.2
- removed net N$30: CV2.3, R2.2
- removed net N$31: CV3.3, R3.2
- removed net N$32: CV4.3, R4.2
- net +5V: no longer R1.1, R2.1, R3.1, R4.1
- net GND: now also CV1.3, CV2.3, CV3.3, CV4.3, DGND3.1; no longer CK_IN.1, CK_IN.3, CK_OUT.1
- net N$19: now also X1.3; no longer MIDI.3
- net N$20: now also X1.4; no longer MIDI.4
Other:
- moved on the sheet: CV1, CV2, CV3, CV4
