File: main_board/main_board.brd (EAGLE design)
At the start: 160 x 100 mm, 142 parts, among them IC1 PIC16F1829SOIC, IC2 V2164, IC3 74HC595D, IC4 TL074D, IC5 TL074D, IC6 TL074D, IC7 74HC14D, IC8 TL074D, IC9 REG1117

Commit message: in work
Parts:
- removed IC7: 74HC14D, 74xx-eu:SO14
- added +5V, AGND1, AGND2, AGND3, AGND4, FR_ATT1, FR_ATT2, FR_ATT3, FR_ATT4, GND21, GND22, TO_ATT1, TO_ATT2, TO_ATT3, TO_ATT4: (no value), pinhead:1X01
- added R55, R56, R57, R58, R59: (no value), rcl:R0805
- C21: device rcl:E2,5-5 -> rcl:C0805
- C24, C25: device rcl:E3,5-10 -> rcl:E2,5-7
- D12, D13: value 1N5819-T -> 1N4004; device diode:DO41-7.6 -> jasons_stuff:DO-VERT
- moved D13 192.9 mm to (116.8, 71.1), flipped to the bottom, turned to 180 degrees
- moved R32 189.1 mm to (109.1, 59.4)
- moved SIGOUT1 186.7 mm to (109.2, 38.7)
- moved SIGIN2 185.5 mm to (100.5, 72.4)
- moved SIGIN1 184.2 mm to (109.2, 36.2)
- moved R31 182.8 mm to (109.1, 57.1)
- moved C11 182.6 mm to (109.1, 48.0)
- moved C7 178.9 mm to (96.4, 61.7), turned to 180 degrees
- moved D12 178.5 mm to (118.1, 43.2), flipped to the bottom
- moved R30 176.7 mm to (109.1, 52.6)
- moved C4 174.3 mm to (102.1, 36.7)
- moved R29 170.2 mm to (109.1, 54.9)
- moved C6 168.3 mm to (91.1, 64.1)
- moved JP1 166.1 mm to (117.6, 57.1), flipped to the bottom, turned to 90 degrees
- moved R18 163.6 mm to (102.1, 44.3)
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Connections:
- removed net 1: D2.A, D6.A, IC7.13, R49.2
- removed net 2: D3.A, D7.A, IC7.11, R50.2
- removed net 3: D4.A, D8.A, IC7.9, R51.2
- removed net 4: D5.A, D9.A, IC7.1, R52.2
- removed net 5: D10.A, D11.A, IC7.3, R53.2
- removed net N$49: IC6.13, IC6.14, IC6.6, IC6.7, IC8.13, IC8.14, IC8.6, IC8.7
- new net N$59: FR_ATT1.1, R14.2
- new net N$60: FR_ATT2.1, R20.2
- new net N$70: FR_ATT3.1, R17.2
- new net N$71: FR_ATT4.1, R23.2
- net +12V: now also C17.1, C19.2, C21.2, D12.A, IC8.4; no longer C21.+, D13.C
- net +5V: now also +5V.1; no longer C17.2, C19.1, IC7.14, IC8.4
- net -12V: now also C17.2, C19.1, C21.1, D13.C, IC8.11; no longer D12.A
- net AGND: now also AGND1.1, AGND2.1, AGND3.1, AGND4.1, C12.1, C13.1, C15.1, C18.1, R35.2, R39.2, R42.2, R45.2
- net CKIN: now also D10.A, D11.A, IC1.19, J1.4, R53.2, R59.2; no longer IC7.4
- net EN_SRC1: now also IC1.10; no longer IC1.6
- net EN_SRC3: now also IC1.6; no longer IC1.10
- net GATE1: now also D2.A, D6.A, IC1.13, R49.2, R55.2; no longer IC1.16, IC7.12
- net GATE2: now also D3.A, D7.A, IC1.14, R50.2, R56.2; no longer IC1.15, IC7.10
- net GATE3: now also D4.A, D8.A, IC1.15, R51.2, R57.2; no longer IC1.14, IC7.8
- net GATE4: now also D5.A, D9.A, IC1.16, R52.2, R58.2; no longer IC1.13, IC7.2
- net GND: now also GND21.1, GND22.1, R55.1, R56.1, R57.1, R58.1, R59.1; no longer C12.1, C13.1, C15.1, C17.1, C18.1, C19.2, C21.-, IC7.5, IC7.7, IC8.11, R35.2, R39.2, R42.2, R45.2
- net N$26: now also TO_ATT1.1; no longer R14.2
- net N$29: now also TO_ATT2.1; no longer R17.2
- net N$32: now also TO_ATT3.1; no longer R20.2
- net N$35: now also TO_ATT4.1; no longer R23.2
- net N$48: now also IC8.3; no longer IC6.5
- net N$50: now also IC6.6, IC6.7; no longer IC6.8, IC6.9
- net N$52: now also IC8.5; no longer IC6.12
- net N$53: now also IC6.8, IC6.9; no longer IC8.1, IC8.2
- net N$55: now also IC8.10; no longer IC8.5
- net N$56: now also IC6.13, IC6.14; no longer IC8.8, IC8.9
- net N$63: now also D13.A; no longer D12.C
- net N$75: now also D12.C; no longer D13.A
- net PWM1: now also IC1.7; no longer IC1.5
- net PWM2: now also IC1.8, IC6.5; no longer IC1.7, IC6.10
- net PWM3: now also IC6.10; no longer IC8.3
- net PWM4: now also IC1.5, IC6.12; no longer IC1.8, IC8.10
- net SWITCH: no longer IC1.19, J1.4
- net VCACV1: now also IC8.1, IC8.2
- net VCACV2: now also IC8.6, IC8.7
- net VCACV3: now also IC8.8, IC8.9
- net VCACV4: now also IC8.13, IC8.14
Routing:
- net +5V: track 0.00 -> 184.8 mm, vias 0 -> 11
- net CKIN: track 0.00 -> 71.9 mm, vias 0 -> 4
- net GATE1: track 0.00 -> 68.8 mm, vias 0 -> 3
- net SWITCH: track 0.00 -> 67.0 mm, vias 0 -> 2
- net GATE3: track 0.00 -> 66.6 mm, vias 0 -> 3
- net GATE2: track 0.00 -> 65.3 mm, vias 0 -> 3
- net PWM3: track 0.00 -> 65.3 mm, vias 0 -> 4
- net GATE4: track 0.00 -> 62.5 mm, vias 0 -> 3
- net KB_READ: track 0.00 -> 60.8 mm, vias 0 -> 2
- net EN_SRC4: track 0.00 -> 60.3 mm
- net N$29: track 0.00 -> 59.0 mm
- net EN_SRC2: track 0.00 -> 58.0 mm, vias 0 -> 2
- net EN_SRC3: track 0.00 -> 58.0 mm, vias 0 -> 2
- net EN_SRC1: track 0.00 -> 53.6 mm, vias 0 -> 2
- net N$32: track 0.00 -> 52.1 mm, vias 0 -> 1
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- added copper zone on layer 1, net AGND
- added copper zone on layer 16, net AGND
- added copper zone on layer 1, net GND
- added copper zone on layer 16, net GND
Other:
- board size 160 x 100 mm -> 107.8 x 40 mm

Commit message: moar stuffs
Parts:
- moved D12 27.9 mm to (118.1, 71.1)
- moved D13 27.9 mm to (116.8, 43.2)
- moved R54 26.9 mm to (71.6, 35.3)
- moved C20 2.68 mm to (68.8, 45.1), turned to 180 degrees
- moved C22 2.01 mm to (67.9, 40.0), turned to 180 degrees
- moved JP1 1.30 mm to (117.3, 55.9), turned to 270 degrees
- moved IC9 1.25 mm to (61.1, 37.6)
- moved C16 1.09 mm to (67.9, 37.7), turned to 180 degrees
- moved C19 0.90 mm to (95.1, 46.0)
Routing:
- net +12V: track 35.9 -> 135.0 mm, vias 4 -> 9
- net -12V: track 36.6 -> 99.5 mm, vias 2 -> 4
- net N$32: track 52.1 -> 77.6 mm, vias 1 -> 2
- net VCAOUT3: track 29.0 -> 46.8 mm
- net +5V: track 184.8 -> 199.8 mm, vias 11 -> 12
- net N$75: track 0.00 -> 13.0 mm
- net N$60: track 21.8 -> 33.9 mm, vias 1 -> 2
- net N$63: track 0.00 -> 10.5 mm
- net GATE1: track 68.8 -> 64.9 mm
- net VCAOUT1: track 30.5 -> 34.2 mm
- net VCACV1: track 27.9 -> 30.9 mm
- net VCACV4: track 28.2 -> 25.9 mm
- net VCAOUT2: track 28.9 -> 31.1 mm
- net GND: track 36.7 -> 34.6 mm, vias 8 -> 10
- net VCACV3: track 27.7 -> 28.9 mm
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
Commit message: and more
Parts:
- moved C5 40.8 mm to (102.1, 36.1), turned to 0 degrees
- moved R19 40.8 mm to (102.1, 38.6), turned to 180 degrees
- moved C4 40.7 mm to (75.9, 67.9), turned to 180 degrees
- moved R16 40.7 mm to (75.9, 70.5), turned to 0 degrees
- moved C17 11.2 mm to (81.4, 58.8)
- moved C21 10.2 mm to (82.7, 72.5)
- moved R21 2.73 mm to (75.9, 62.9)
- moved R20 2.73 mm to (75.9, 65.4)
- moved IC5 2.29 mm to (82.8, 66.7)
- moved R23 1.89 mm to (89.7, 67.9)
- moved C6 1.89 mm to (89.7, 62.9)
- moved R22 1.89 mm to (89.7, 65.4)
- moved R24 1.89 mm to (89.7, 70.5)
- moved D12 0.76 mm to (117.3, 71.1)
- moved D13 0.76 mm to (116.1, 43.2)
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Connections:
- net N$26 renamed TO_ATT1
- net N$35 renamed TO_ATT4
- net N$59 renamed FR_ATT1
- removed net N$29: C4.2, IC4.8, R16.1, TO_ATT2.1
- removed net N$32: C5.2, IC5.1, R19.1, TO_ATT3.1
- new net TO_ATT2: C4.2, IC5.1, R16.1, TO_ATT2.1
- new net TO_ATT3: C5.2, IC4.8, R19.1, TO_ATT3.1
- net N$31: now also SIGOUT3.1; no longer SIGOUT2.1
- net N$34: now also SIGOUT2.1; no longer SIGOUT3.1
- net VCAOUT2: now also IC5.3; no longer IC4.10
- net VCAOUT3: now also IC4.10; no longer IC5.3
Routing:
- net N$32: track 77.6 -> 0.00 mm, vias 2 -> 0
- net N$29: track 60.2 -> 0.00 mm
- net N$34: track 24.4 -> 68.0 mm, vias 0 -> 2
- net TO_ATT2: track 0.00 -> 34.8 mm, vias 0 -> 2
- net TO_ATT3: track 0.00 -> 24.1 mm
- net N$31: track 19.0 -> 42.6 mm
- net AGND: track 18.6 -> 0.00 mm, vias 16 -> 18
- net VCAOUT3: track 46.8 -> 29.6 mm
- net VCAOUT2: track 31.1 -> 44.8 mm, vias 2 -> 4
- net +12V: track 135.0 -> 142.4 mm, vias 9 -> 3
- net TO_ATT1: track 41.9 -> 37.1 mm, vias 0 -> 3
- net VCACV2: track 27.9 -> 32.7 mm
- net N$39: track 41.6 -> 37.3 mm, vias 1 -> 2
- net N$45: track 33.1 -> 29.7 mm
- net N$37: track 12.3 -> 15.7 mm
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
Commit message: MORE
Parts:
- removed C25: (no value), rcl:E2,5-7
- removed OK1: 6N138, optocoupler:DIL08
- removed U$1: 0805DIODE, jasons_stuff:0805DIODE
- added D14: (no value), diode:SOD123
- added F1, F2: (no value), adafruit:R1206
- added IC7: TL074D, linear:SO14
- added L1, L2: (no value), wuerth-elektronik:0805
- added R60: (no value), rcl:R0805
- C20: device rcl:E2,5-5 -> rcl:C0805
- C22, C23: device rcl:C0805 -> rcl:E2,5-7
- C24: device rcl:E2,5-7 -> rcl:E2,5-5
- D11: value (none) -> 0805DIODE; device microbuilder:SOD-123 -> jasons_stuff:0805DIODE
- D12: value 1N4004 -> (none); device jasons_stuff:DO-VERT -> microbuilder:SOD-123
- D13: value 1N4004 -> (none); device jasons_stuff:DO-VERT -> diode:SOD123
- IC1: value PIC16F1829SOIC -> 74HC595D; device jason_eagle6:SO20W -> 74xx-eu:SO16
- IC2: value V2164 -> TL074D; device jason_eagle6:SO16 -> linear:SO14
- IC3: value 74HC595D -> PIC16F1829SOIC; device 74xx-eu:SO16 -> jason_eagle6:SO20W
- IC6: value TL074D -> V2164; device linear:SO14 -> jason_eagle6:SO16
- IC8: value TL074D -> REG1117; device linear:SO14 -> burr-brown:SOT223
- IC9: value REG1117 -> 6N138; device burr-brown:SOT223 -> optocoupler:DIL08
- R25: device rcl:R0805 -> rcl:C0805
- moved R52 90.7 mm to (109.1, 57.1), turned to 0 degrees
- moved R51 88.6 mm to (109.1, 59.4), turned to 0 degrees
- moved R59 88.5 mm to (102.1, 41.1)
- moved D1 88.5 mm to (21.6, 58.3), turned to 0 degrees
- moved R58 87.1 mm to (102.1, 43.7)
- moved R53 80.3 mm to (109.1, 54.9), turned to 0 degrees
- moved R57 74.5 mm to (88.0, 36.1), turned to 180 degrees
- moved R56 74.4 mm to (88.0, 38.6), turned to 180 degrees
- moved R55 74.3 mm to (88.0, 41.1)
- moved R50 72.4 mm to (96.4, 52.6), turned to 180 degrees
- moved R49 70.3 mm to (96.4, 54.9), turned to 180 degrees
- moved R17 69.2 mm to (38.1, 67.6)
- moved R19 68.5 mm to (38.1, 63.0), turned to 0 degrees
- moved R18 67.6 mm to (38.1, 65.3)
- moved R26 62.2 mm to (38.1, 37.8), turned to 0 degrees
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- renumbered T1 to Q3, T2 to Q2, T3 to Q1, T4 to Q4
Connections:
- new net N$32: D13.C, F1.1, L1.2
- new net N$35: D14.A, F2.1, L2.2
- net +12V: now also C15.1, C22.+, C3.2, C6.2, C7.1, IC6.16, IC7.4, IC8.3, L1.1, R46.2; no longer C17.1, C2.1, C21.2, C22.2, C24.+, D12.A, IC2.16, IC8.4, IC9.3, R33.2
- net +5V: now also C2.2, C24.+, C4.2, D10.C, D6.C, D7.C, D8.C, D9.C, IC1.10, IC1.16, IC2.4, IC3.1, IC8.2, IC9.8, R25.2, R28.2; no longer C14.2, C16.2, C20.+, C23.2, D11.C, D2.C, D3.C, D4.C, D5.C, IC1.1, IC3.10, IC3.16, IC6.4, IC9.2, OK1.8, R48.2
- net -12V: now also C23.-, C6.1, C7.2, D12.A, IC6.9, IC7.11, L2.1; no longer C11.1, C17.2, C25.-, D1.A, D13.C, IC2.9, IC8.11
- net AGND: now also C11.1, C14.1, C15.2, C16.1, C17.1, C21.2, C22.-, C23.+, D12.C, D13.A, D14.C, IC6.8, IC7.13, IC7.2, IC7.6, IC7.9, R31.1, R38.2, R41.2; no longer C10.1, C11.2, C15.1, C18.1, C2.2, C24.-, C25.+, C7.1, D1.C, IC2.8, IC5.13, IC5.2, IC5.6, IC5.9, R35.2, R39.2, R54.1
- net CKIN: now also D1.A, D6.A, IC3.19, R14.2, R5.2; no longer D10.A, D11.A, IC1.19, R53.2, R59.2
- net EN_SRC1: now also IC3.10, R3.2; no longer IC1.10, R9.2
- net EN_SRC2: now also IC3.9, R2.2; no longer IC1.9, R10.2
- net EN_SRC3: now also IC3.6, R1.2; no longer IC1.6, R11.2
- net EN_SRC4: now also IC1.14, IC3.11, R4.2; no longer IC1.11, IC3.14, R12.2
- net FR_ATT1: now also R56.2; no longer R14.2
- net GATE1: now also D7.A, IC3.13, R13.2, R6.2; no longer D6.A, IC1.13, R49.2, R55.2
- net GATE2: now also D8.A, IC3.14, R12.2, R7.2; no longer D7.A, IC1.14, R50.2, R56.2
- net GATE3: now also D9.A, IC3.15, R11.2, R8.2; no longer D8.A, IC1.15, R51.2, R57.2
- net GATE4: now also D10.A, IC3.16, R10.2, R9.2; no longer D9.A, IC1.16, R52.2, R58.2
- net GND: now also C2.1, C24.-, C3.1, C4.1, D1.C, D2.C, D3.C, D4.C, D5.C, IC1.13, IC1.8, IC2.11, IC3.20, IC8.1, IC9.5, R25.1, R30.2, R31.2, R5.1, R6.1, R7.1, R8.1, R9.1; no longer C14.1, C16.1, C20.-, C22.1, C23.1, D10.C, D6.C, D7.C, D8.C, D9.C, IC1.20, IC3.13, IC3.8, IC6.11, IC9.1, OK1.5, R47.2, R54.2, R55.1, R56.1, R57.1, R58.1, R59.1
- net KB_READ: now also IC3.18; no longer IC1.18
- net MIDI_RX: now also IC3.12, IC9.6, R28.1; no longer IC1.12, OK1.6, R48.1
- net N$1: now also IC1.7, R22.2; no longer IC3.7, R1.2
- net N$10: now also R21.1; no longer R2.1
- net N$11: now also R20.1; no longer R3.1
- net N$12: now also R19.1; no longer R4.1
- net N$13: now also R18.1; no longer R5.1
- net N$14: now also R17.1; no longer R6.1
- net N$15: now also R16.1; no longer R7.1
- net N$16: now also R15.1; no longer R8.1
- net N$2: now also IC1.6, R21.2; no longer IC3.6, R2.2
- net N$21: now also IC6.1, R46.1; no longer IC2.1, R33.1
- net N$22: now also R3.1; no longer R9.1
- net N$23: now also R2.1; no longer R10.1
- net N$24: now also R1.1; no longer R11.1
- net N$25: now also R4.1; no longer R12.1
- net N$27: now also IC7.5, R56.1, R57.2; no longer IC4.5, R14.1, R15.2
- net N$28: now also IC7.7, R57.1; no longer IC4.7, R15.1
- net N$3: now also IC1.5, R20.2; no longer IC3.5, R3.2
- net N$30: now also IC7.12, R58.2, R59.1; no longer IC4.12, R17.1, R18.2
- net N$31: now also IC7.14, R58.1; no longer IC4.14, R18.1
- net N$33: now also IC4.5, R33.1, R34.2; no longer IC5.5, R20.1, R21.2
- net N$34: now also IC4.7, R34.1; no longer IC5.7, R21.1
- net N$36: now also IC4.12, R35.2, R36.1; no longer IC5.12, R23.1, R24.2
- net N$37: now also IC4.14, R35.1; no longer IC5.14, R24.1
- net N$38: now also C13.2, R47.2; no longer C7.2, R26.2
- net N$39: now also R48.2; no longer R25.2
- net N$4: now also IC1.4, R19.2; no longer IC3.4, R4.2
- net N$40: now also C14.2, R50.2; no longer C8.2, R28.2
- net N$41: now also R49.2; no longer R27.2
- net N$42: now also C17.2, R54.2; no longer C9.2, R30.2
- net N$43: now also R53.2; no longer R29.2
- net N$44: now also C16.2, R51.2; no longer C10.2, R32.2
- net N$45: now also R52.2; no longer R31.2
- net N$46: now also R24.1; no longer R34.1
- net N$47: now also IC2.1, IC2.2, R24.2; no longer IC6.1, IC6.2, R34.2
- net N$48: now also C8.2, IC5.3, R38.1, R39.2; no longer C12.2, IC8.3, R35.1, R38.2
- net N$5: now also IC1.3, R18.2; no longer IC3.3, R5.2
- net N$50: now also IC2.6, IC2.7, R27.2; no longer IC6.6, IC6.7, R36.2
- net N$51: now also R27.1; no longer R36.1
- net N$52: now also C9.2, IC5.5, R40.2, R41.1; no longer C13.2, IC8.5, R37.2, R39.1
- net N$53: now also IC2.8, IC2.9, R26.2; no longer IC6.8, IC6.9, R40.2
- net N$54: now also R26.1; no longer R40.1
- net N$55: now also C12.2, IC5.10, R44.2, R45.1; no longer C15.2, IC8.10, R41.2, R42.1
- net N$56: now also IC2.13, IC2.14, R23.2; no longer IC6.13, IC6.14, R43.2
- net N$57: now also R23.1; no longer R43.1
- net N$58: now also C11.2, IC5.12, R42.1, R43.2; no longer C18.2, IC8.12, R44.2, R45.1
- net N$6: now also IC1.2, R17.2; no longer IC3.2, R6.2
- net N$60: now also R33.2; no longer R20.2
- net N$61: now also R13.1; no longer R49.1
- net N$62: now also IC9.7, R30.1; no longer OK1.7, R47.1
- net N$63: now also F2.2; no longer D13.A
- net N$64: now also D11.A, IC9.2, R29.2; no longer OK1.2, R46.2, U$1.A
- net N$65: now also D11.C, IC9.3; no longer OK1.3, U$1.C
- net N$66: now also R29.1; no longer R46.1
- net N$67: now also R12.1; no longer R50.1
- net N$68: now also R11.1; no longer R51.1
- net N$69: now also R10.1; no longer R52.1
- net N$7: now also IC1.1, R16.2; no longer IC3.1, R7.2
- net N$70: now also R59.2; no longer R17.2
- net N$71: now also R36.2; no longer R23.2
- net N$74: now also R14.1; no longer R53.1
- net N$75: now also F1.2; no longer D12.C
- net N$8: now also IC1.15, R15.2; no longer IC3.15, R8.2
- net N$9: now also R22.1; no longer R1.1
- net PWM1: now also IC2.3, IC3.7, R39.1; no longer IC1.7, IC6.3, R38.1
- net PWM2: now also IC2.5, IC3.8, R40.1; no longer IC1.8, IC6.5, R37.1
- net PWM3: now also IC2.10, IC3.17, R44.1; no longer IC1.17, IC6.10, R41.1
- net PWM4: now also IC2.12, IC3.5, R43.1; no longer IC1.5, IC6.12, R44.1
- net SR_RCK: now also IC1.12, IC3.2; no longer IC1.2, IC3.12
- net SR_SCK: now also IC1.11, IC3.3; no longer IC1.3, IC3.11
- net SWITCH: now also IC3.4; no longer IC1.4
- net TO_ATT1: now also C18.2, IC7.1, R55.1; no longer C3.2, IC4.1, R13.1
- net TO_ATT2: now also C5.2, IC4.1, R32.1; no longer C4.2, IC5.1, R16.1
- net TO_ATT3: now also C20.2, IC7.8, R60.1; no longer C5.2, IC4.8, R19.1
- net TO_ATT4: now also C10.2, IC4.8, R37.1; no longer C6.2, IC5.8, R22.1
- net VCACV1: now also IC5.1, IC5.2, IC6.3; no longer IC2.3, IC8.1, IC8.2
- net VCACV2: now also IC5.6, IC5.7, IC6.6; no longer IC2.6, IC8.6, IC8.7
- net VCACV3: now also IC5.8, IC5.9, IC6.11; no longer IC2.11, IC8.8, IC8.9
- net VCACV4: now also IC5.13, IC5.14, IC6.14; no longer IC2.14, IC8.13, IC8.14
- net VCAIN1: now also IC6.2, R47.1, R48.1; no longer IC2.2, R25.1, R26.1
- net VCAIN2: now also IC6.7, R49.1, R50.1; no longer IC2.7, R27.1, R28.1
- net VCAIN3: now also IC6.10, R53.1, R54.1; no longer IC2.10, R29.1, R30.1
- net VCAIN4: now also IC6.15, R51.1, R52.1; no longer IC2.15, R31.1, R32.1
- net VCAOUT1: now also C18.1, IC6.4, IC7.3, R55.2; no longer C3.1, IC2.4, IC4.3, R13.2
- net VCAOUT2: now also C5.1, IC4.3, IC6.5, R32.2; no longer C4.1, IC2.5, IC5.3, R16.2
- net VCAOUT3: now also C20.1, IC6.12, IC7.10, R60.2; no longer C5.1, IC2.12, IC4.10, R19.2
- net VCAOUT4: now also C10.1, IC4.10, IC6.13, R37.2; no longer C6.1, IC2.13, IC5.10, R22.2
Routing:
- net N$35: track 0.00 -> 7.25 mm
- net N$75: track 12.7 -> 5.65 mm
- net N$32: track 0.00 -> 5.61 mm
- net N$63: track 10.2 -> 5.52 mm
- net -12V: track 97.1 -> 98.6 mm, vias 3 -> 4
- net +12V: track 142.4 -> 141.9 mm, vias 3 -> 4

Commit message: more
Parts:
- removed D13, D14: (no value), diode:SOD123
- added C25, C26, C27: (no value), rcl:C0805
- added D15, D16: 1N4004, jasons_stuff:DO-VERT
- F1, F2: device adafruit:R1206 -> microbuilder:PTC1210
- moved C7 16.4 mm to (80.0, 42.4), turned to 270 degrees
- moved C6 12.3 mm to (79.9, 60.6), turned to 0 degrees
- moved C19 3.43 mm to (92.2, 45.6), turned to 0 degrees
- moved L2 1.15 mm to (117.0, 43.1), turned to 90 degrees
- moved L1 0.77 mm to (117.5, 68.3)
- moved F1 0.52 mm to (117.5, 64.5), turned to 90 degrees
- moved F2 0.51 mm to (117.3, 47.4), turned to 270 degrees
- renumbered AGND1 to +12V, AGND3 to -12V, J1 to ICSP, JP1 to POWER
Connections:
- net +12V: now also +12V.1
- net -12V: now also -12V.1, C25.2, C26.2, C27.1; no longer C19.1, C6.1, C7.2
- net AGND: now also C19.1, C25.1, C26.1, C27.2, C6.1, C7.2, D15.A, D16.C; no longer +12V.1, -12V.1, D13.A, D14.C
- net N$32: now also D15.C, F1.P$2; no longer D13.C, F1.1
- net N$35: now also D16.A, F2.P$2; no longer D14.A, F2.1
- net N$63: now also F2.P$1; no longer F2.2
- net N$75: now also F1.P$1; no longer F1.2
Routing:
- net -12V: track 98.6 -> 108.6 mm
- net TO_ATT1: track 37.1 -> 33.4 mm
- net +12V: track 141.9 -> 145.3 mm, vias 4 -> 5
- net N$35: track 7.25 -> 4.27 mm
- net VCACV2: track 32.7 -> 31.2 mm
- net VCAOUT2: track 44.8 -> 43.5 mm
- net N$75: track 5.65 -> 4.65 mm
- net N$63: track 5.52 -> 4.57 mm
- net N$32: track 5.61 -> 6.52 mm
- net VCAOUT1: track 32.1 -> 32.7 mm
Other:
- board text added: "-12V"
- board text added: "DIGITALLY CONTROLLED QUAD VCA/MIXER"
- board text added: "MAIN BOARD V1"
- board text added: "hotchk155"

Commit message: fixes
Parts:
- added D13, D14, D17, D18, D19, D20, D21, D22: 0805DIODE, jasons_stuff:0805DIODE
- moved R31 13.3 mm to (71.8, 48.6), flipped to the bottom, turned to 0 degrees
- moved R28 11.8 mm to (67.7, 59.4), turned to 180 degrees
- moved R30 9.48 mm to (67.7, 72.5), turned to 0 degrees
- moved C1 6.84 mm to (56.1, 70.6), turned to 270 degrees
- moved C22 6.67 mm to (73.5, 38.7), flipped to the top, turned to 90 degrees
- moved D11 6.08 mm to (61.8, 59.4), turned to 180 degrees
- moved C23 5.78 mm to (81.3, 38.7), flipped to the top, turned to 90 degrees
- moved R22 4.42 mm to (42.3, 57.5)
- moved R21 4.38 mm to (42.3, 59.7)
- moved R20 4.34 mm to (42.3, 61.8)
- moved R19 4.31 mm to (42.3, 64.0)
- moved R18 4.28 mm to (42.3, 66.2)
- moved R17 4.26 mm to (42.3, 68.3)
- moved R16 4.24 mm to (42.3, 70.5)
- moved R15 4.22 mm to (42.3, 72.6)
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Connections:
- new net N$26: D13.C, SINK8.1
- new net N$29: D14.C, SINK7.1
- new net N$49: D17.C, SINK6.1
- new net N$59: D18.C, SINK5.1
- new net N$72: D19.C, SINK4.1
- new net N$73: D20.C, SINK3.1
- new net N$76: D21.C, SINK2.1
- new net N$77: D22.C, SINK1.1
- net AGND: now also IC4.10, IC4.12, IC4.3, IC4.5, IC7.10, IC7.12, IC7.3, IC7.5; no longer IC4.13, IC4.2, IC4.6, IC4.9, IC7.13, IC7.2, IC7.6, IC7.9
- net CKIN: now also D1.C; no longer D1.A
- net GATE1: now also D2.C; no longer D2.A
- net GATE2: now also D3.C; no longer D3.A
- net GATE3: now also D4.C; no longer D4.A
- net GATE4: now also D5.C; no longer D5.A
- net GND: now also D1.A, D2.A, D3.A, D4.A, D5.A; no longer D1.C, D2.C, D3.C, D4.C, D5.C
- net N$10: now also D14.A; no longer SINK7.1
- net N$11: now also D17.A; no longer SINK6.1
- net N$12: now also D18.A; no longer SINK5.1
- net N$13: now also D19.A; no longer SINK4.1
- net N$14: now also D20.A; no longer SINK3.1
- net N$15: now also D21.A; no longer SINK2.1
- net N$16: now also D22.A; no longer SINK1.1
- net N$27: now also IC7.6; no longer IC7.5
- net N$30: now also IC7.13; no longer IC7.12
- net N$33: now also IC4.6; no longer IC4.5
- net N$36: now also IC4.13; no longer IC4.12
- net N$9: now also D13.A; no longer SINK8.1
- net VCAOUT1: now also IC7.2; no longer IC7.3
- net VCAOUT2: now also IC4.2; no longer IC4.3
- net VCAOUT3: now also IC7.9; no longer IC7.10
- net VCAOUT4: now also IC4.9; no longer IC4.10
Routing:
- net N$26: track 0.00 -> 36.2 mm, vias 0 -> 1
- net +5V: track 199.8 -> 234.4 mm, vias 12 -> 13
- net N$49: track 0.00 -> 33.7 mm, vias 0 -> 1
- net N$29: track 0.00 -> 30.8 mm, vias 0 -> 1
- net N$9: track 30.7 -> 2.49 mm, vias 1 -> 0
- net N$10: track 24.3 -> 2.49 mm, vias 1 -> 0
- net N$72: track 0.00 -> 20.3 mm, vias 0 -> 1
- net N$11: track 22.3 -> 2.49 mm, vias 1 -> 0
- net N$59: track 0.00 -> 18.3 mm, vias 0 -> 1
- net N$13: track 18.4 -> 2.49 mm, vias 1 -> 0
- net N$12: track 16.9 -> 2.49 mm, vias 1 -> 0
- net GND: track 34.6 -> 22.7 mm, vias 10 -> 11
- net N$77: track 0.00 -> 11.5 mm
- net N$73: track 0.00 -> 11.1 mm, vias 0 -> 1
- net N$64: track 5.54 -> 16.0 mm
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