File: main_board/main_board.brd (EAGLE design)
At the start: 107.8 x 40 mm, 176 parts, among them IC1 74HC595D, IC2 TL074D, IC3 PIC16F1829SOIC, IC4 TL074D, IC5 TL074D, IC6 V2164, IC7 TL074D, IC8 REG1117, IC9 6N138

Commit message: fixes
Parts:
- D15, D16: value 1N4004 -> MBR0520LT; device jasons_stuff:DO-VERT -> diode:SOD123
- moved L2 1.61 mm to (117.5, 41.5), turned to 0 degrees
- moved D15 1.37 mm to (116.7, 70.9), flipped to the top, turned to 180 degrees
- moved D16 1.02 mm to (116.6, 43.6), flipped to the top
Routing:
- net -12V: track 103.1 -> 106.4 mm
- net N$35: track 4.27 -> 5.41 mm
- net N$32: track 6.52 -> 5.43 mm
Changed lines of the file:
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@@
 <attribute name="VALUE" x="113.538" y="49.911" size="1.27" layer="27" rot="R270"/>
 </element>
-<element name="D15" library="jasons_stuff" package="DO-VERT" value="1N4004" x="117.475" y="72.009" smashed="yes" rot="MR0">
-<attribute name="NAME" x="113.665" y="71.501" size="1.27" layer="26" ratio="10" rot="MR0"/>
+<element name="L1" library="wuerth-elektronik" package="0805" value="" x="117.475" y="68.326" smashed="yes">
+<attribute name="VALUE" x="115.57" y="69.2785" size="0.6096" layer="27"/>
+<attribute name="NAME" x="113.665" y="67.8815" size="1.27" layer="25"/>
 </element>
-<element name="D16" library="jasons_stuff" package="DO-VERT" value="1N4004" x="117.602" y="43.561" smashed="yes" rot="MR0">
-<attribute name="NAME" x="114.046" y="42.926" size="1.27" layer="26" ratio="10" rot="MR0"/>
-</element>
-<element name="L1" library="wuerth-elektronik" package="0805" value="" x="117.475" y="68.326"/>
-<element name="L2" library="wuerth-elektronik" package="0805" value="" x="116.967" y="43.053" smashed="yes" rot="R90">
-<attribute name="VALUE" x="116.0145" y="41.148" size="0.6096" layer="27" rot="R90"/>
-<attribute name="NAME" x="118.5545" y="41.148" size="0.6096" layer="25" rot="R90"/>
+<element name="L2" library="wuerth-elektronik" package="0805" value="" x="117.475" y="41.529" smashed="yes">
+<attribute name="VALUE" x="115.57" y="42.4815" size="0.6096" layer="27"/>
+<attribute name="NAME" x="112.014" y="40.3225" size="1.27" layer="25"/>
 </element>
 <element name="D13" library="jasons_stuff" package="0805DIODE" value="0805DIODE" x="37.592" y="57.531" smashed="yes" rot="R180">
@@
 <element name="D22" library="jasons_stuff" package="0805DIODE" value="0805DIODE" x="37.719" y="72.644" smashed="yes" rot="R180">
 <attribute name="NAME" x="38.6158" y="56.304" size="1.27" layer="21" rot="R180"/>
+</element>
+<element name="D15" library="diode" package="SOD123" value="MBR0520LT" x="116.713" y="70.866" smashed="yes" rot="R180">
+<attribute name="NAME" x="113.495" y="71.39" size="1.27" layer="25" rot="R180"/>
+</element>
+<element name="D16" library="diode" package="SOD123" value="MBR0520LT" x="116.586" y="43.561" smashed="yes">
+<attribute name="NAME" x="110.533" y="42.021" size="1.27" layer="25"/>
 </element>
 </elements>
@@
 <contactref element="C7" pad="2"/>
 <contactref element="C27" pad="2"/>
-<contactref element="D15" pad="A"/>
-<contactref element="D16" pad="C"/>
 <contactref element="IC7" pad="3"/>
 <contactref element="IC4" pad="3"/>
@@
 <contactref element="IC7" pad="12"/>
 <contactref element="IC4" pad="12"/>
+<contactref element="D16" pad="C"/>
+<contactref element="D15" pad="A"/>
 </signal>
 <signal name="TO_ATT2">
@@
 <wire x1="107.315" y1="45.792" x2="107.315" y2="43.18" width="0.3048" layer="1"/>
 <via x="107.315" y="43.18" extent="1-16" drill="0.6"/>
-<via x="114.935" y="41.402" extent="1-16" drill="0.6"/>
 <contactref element="-12V" pad="1"/>
-<wire x1="118.11" y1="40.81" x2="118.11" y2="37.465" width="0.3048" layer="1"/>
-<wire x1="118.11" y1="37.465" x2="116.84" y2="36.195" width="0.3048" layer="1"/>
 <contactref element="C26" pad="2"/>
 <contactref element="C25" pad="2"/>
@@
 <wire x1="82.677" y1="47.244" x2="82.169" y2="47.752" width="0.3048" layer="1"/>
 <contactref element="L2" pad="1"/>
-<wire x1="114.935" y1="41.402" x2="116.416" y2="41.402" width="0.6096" layer="1"/>
-<wire x1="116.416" y1="41.402" x2="116.967" y2="41.953" width="0.6096" layer="1"/>
-<wire x1="118.11" y1="40.81" x2="116.967" y2="41.953" width="0.3048" layer="1"/>
 <wire x1="107.315" y1="43.18" x2="108.458" y2="43.18" width="0.6096" layer="16"/>
-<wire x1="108.458" y1="43.18" x2="110.236" y2="41.402" width="0.6096" layer="16"/>
-<wire x1="110.236" y1="41.402" x2="114.935" y2="41.402" width="0.6096" layer="16"/>
 <wire x1="95.758" y1="45.212" x2="82.677" y2="45.212" width="0.6096" layer="16"/>
 <wire x1="82.677" y1="45.212" x2="82.677" y2="46.863" width="0.6096" layer="16"/>
@@
 <wire x1="81.28" y1="40.005" x2="82.677" y2="41.402" width="0.6096" layer="16"/>
 <wire x1="82.677" y1="41.402" x2="82.677" y2="45.212" width="0.6096" layer="16"/>
+<wire x1="116.84" y1="36.195" x2="118.491" y2="36.195" width="0.6096" layer="16"/>
+<wire x1="118.491" y1="36.195" x2="118.618" y2="36.322" width="0.6096" layer="16"/>
+<wire x1="118.618" y1="36.322" x2="118.618" y2="41.529" width="0.6096" layer="16"/>
+<wire x1="108.458" y1="43.18" x2="110.109" y2="41.529" width="0.6096" layer="16"/>
+<wire x1="110.109" y1="41.529" x2="113.03" y2="41.529" width="0.6096" layer="16"/>
+<wire x1="114.808" y1="41.529" x2="118.618" y2="41.529" width="0.6096" layer="16"/>
+<wire x1="116.375" y1="41.529" x2="114.808" y2="41.529" width="0.6096" layer="1"/>
+<via x="114.808" y="41.529" extent="1-16" drill="0.6"/>
+<wire x1="114.808" y1="41.529" x2="113.03" y2="41.529" width="0.6096" layer="16"/>
 </signal>
 <signal name="+12V">
@@
 <signal name="N$32">
 <contactref element="F1" pad="P$2"/>
-<contactref element="D15" pad="C"/>
 <contactref element="L1" pad="2"/>
-<wire x1="118.745" y1="72.009" x2="118.745" y2="68.496" width="0.6096" layer="1"/>
 <wire x1="118.745" y1="68.496" x2="118.575" y2="68.326" width="0.6096" layer="1"/>
 <wire x1="118.575" y1="68.326" x2="118.575" y2="67.116" width="0.6096" layer="1"/>
 <wire x1="118.575" y1="67.116" x2="117.475" y2="66.016" width="0.6096" layer="1"/>
+<contactref element="D15" pad="C"/>
+<wire x1="118.745" y1="68.496" x2="118.613" y2="68.628" width="0.6096" layer="1"/>
+<wire x1="118.613" y1="68.628" x2="118.613" y2="70.866" width="0.6096" layer="1"/>
 </signal>
 <signal name="N$35">
 <contactref element="F2" pad="P$2"/>
-<contactref element="D16" pad="A"/>
 <contactref element="L2" pad="2"/>
-<wire x1="116.967" y1="44.153" x2="116.967" y2="45.593" width="0.6096" layer="1"/>
 <wire x1="116.967" y1="45.593" x2="116.84" y2="45.72" width="0.6096" layer="1"/>
-<wire x1="116.967" y1="44.153" x2="115.654" y2="44.153" width="0.6096" layer="1"/>
-<wire x1="115.654" y1="44.153" x2="115.062" y2="43.561" width="0.6096" layer="1"/>
 <wire x1="117.348" y1="45.871" x2="117.245" y2="45.871" width="0.6096" layer="1"/>
 <wire x1="117.245" y1="45.871" x2="116.967" y2="45.593" width="0.6096" layer="1"/>
+<contactref element="D16" pad="A"/>
+<wire x1="116.967" y1="45.593" x2="118.486" y2="44.074" width="0.6096" layer="1"/>
+<wire x1="118.486" y1="44.074" x2="118.486" y2="43.561" width="0.6096" layer="1"/>
+<wire x1="118.486" y1="43.561" x2="118.575" y2="43.472" width="0.6096" layer="1"/>
+<wire x1="118.575" y1="43.472" x2="118.575" y2="41.529" width="0.6096" layer="1"/>
 </signal>
 <signal name="N$9">

Commit message: fixes
Parts:
- removed D1, D6: (no value), microbuilder:SOD-123
- removed R14, R5: (no value), rcl:R0805
- turned GND1 to 0 degrees
- renumbered CLOCKIN to GND1
Connections:
- removed net N$74: GND1.1, R14.1
- net +5V: no longer D6.C
- net CKIN: no longer D1.C, D6.A, R14.2, R5.2
- net GND: now also GND1.1; no longer D1.A, R5.1
Routing:
- net CKIN: track 71.9 -> 3.35 mm, vias 4 -> 1
- net GND: track 22.7 -> 18.5 mm
- net N$74: track 3.51 -> 0.00 mm
