File: main_board/main_board.sch (EAGLE design)
At the start: 142 parts, among them IC1 PIC16F1829SOIC, IC2 V2164, IC3 74HC595D, IC4 TL074D, IC5 TL074D, IC6 TL074D, IC7 74HC14D, IC8 TL074D, IC9 REG1117

Commit message: in work
Parts:
- removed IC7: 74HC14D, 74xx-eu:74HC14D
- added +5V, AGND1, AGND2, AGND3, AGND4, FR_ATT1, FR_ATT2, FR_ATT3, FR_ATT4, GND21, GND22, TO_ATT1, TO_ATT2, TO_ATT3, TO_ATT4: (no value), pinhead:PINHD-1X1
- added R55, R56, R57, R58, R59: (no value), rcl:R-EU_R0805
- C21: device rcl:CPOL-EUE2.5-5 -> rcl:C-EUC0805
- C24, C25: device rcl:CPOL-EUE3.5-10 -> rcl:CPOL-EUE2.5-7
- D12, D13: value 1N5819-T -> 1N4004; device diode:1N5819-T -> jasons_stuff:1N4004
Connections:
- removed net 1: D2.A, D6.A, IC7A.I, R49.2
- removed net 2: D3.A, D7.A, IC7B.I, R50.2
- removed net 3: D4.A, D8.A, IC7C.I, R51.2
- removed net 4: D5.A, D9.A, IC7D.I, R52.2
- removed net 5: D10.A, D11.A, IC7E.I, R53.2
- removed net N$49: IC6B.-IN, IC6B.OUT, IC6D.-IN, IC6D.OUT, IC8B.-IN, IC8B.OUT, IC8D.-IN, IC8D.OUT
- new net N$59: FR_ATT1.1, R14.2
- new net N$60: FR_ATT2.1, R20.2
- new net N$70: FR_ATT3.1, R17.2
- new net N$71: FR_ATT4.1, R23.2
- net +12V: now also C17.1, C19.2, C21.2, D12.A, IC8P.V+; no longer C21.+, D13.C
- net +5V: now also +5V.1; no longer C17.2, C19.1, IC7P.VCC, IC8P.V+
- net -12V: now also C17.2, C19.1, C21.1, D13.C, IC8P.V-; no longer D12.A
- net AGND: now also AGND1.1, AGND2.1, AGND3.1, AGND4.1, C12.1, C13.1, C15.1, C18.1, R35.2, R39.2, R42.2, R45.2
- net CKIN: now also D10.A, D11.A, IC1.RA0, J1.ICSP_DAT/PGD, R53.2, R59.2; no longer IC7E.O
- net EN_SRC1: now also IC1.RB7; no longer IC1.RC4
- net EN_SRC3: now also IC1.RC4; no longer IC1.RB7
- net GATE1: now also D2.A, D6.A, IC1.RB4, R49.2, R55.2; no longer IC1.RC0, IC7A.O
- net GATE2: now also D3.A, D7.A, IC1.RC2, R50.2, R56.2; no longer IC1.RC1, IC7B.O
- net GATE3: now also D4.A, D8.A, IC1.RC1, R51.2, R57.2; no longer IC1.RC2, IC7C.O
- net GATE4: now also D5.A, D9.A, IC1.RC0, R52.2, R58.2; no longer IC1.RB4, IC7D.O
- net GND: now also GND21.1, GND22.1, R55.1, R56.1, R57.1, R58.1, R59.1; no longer C12.1, C13.1, C15.1, C17.1, C18.1, C19.2, C21.-, IC7F.I, IC7P.GND, IC8P.V-, R35.2, R39.2, R42.2, R45.2
- net N$26: now also TO_ATT1.1; no longer R14.2
- net N$29: now also TO_ATT2.1; no longer R17.2
- net N$32: now also TO_ATT3.1; no longer R20.2
- net N$35: now also TO_ATT4.1; no longer R23.2
- net N$48: now also IC8A.+IN; no longer IC6B.+IN
- net N$50: now also IC6B.-IN, IC6B.OUT; no longer IC6C.-IN, IC6C.OUT
- net N$52: now also IC8B.+IN; no longer IC6D.+IN
- net N$53: now also IC6C.-IN, IC6C.OUT; no longer IC8A.-IN, IC8A.OUT
- net N$55: now also IC8C.+IN; no longer IC8B.+IN
- net N$56: now also IC6D.-IN, IC6D.OUT; no longer IC8C.-IN, IC8C.OUT
- net N$63: now also D13.A; no longer D12.C
- net N$75: now also D12.C; no longer D13.A
- net PWM1: now also IC1.RC3; no longer IC1.RC5
- net PWM2: now also IC1.RC6, IC6B.+IN; no longer IC1.RC3, IC6C.+IN
- net PWM3: now also IC6C.+IN; no longer IC8A.+IN
- net PWM4: now also IC1.RC5, IC6D.+IN; no longer IC1.RC6, IC8C.+IN
- net SWITCH: no longer IC1.RA0, J1.ICSP_DAT/PGD
- net VCACV1: now also IC8A.-IN, IC8A.OUT
- net VCACV2: now also IC8B.-IN, IC8B.OUT
- net VCACV3: now also IC8C.-IN, IC8C.OUT
- net VCACV4: now also IC8D.-IN, IC8D.OUT
Other:
- note removed: "VCA OUTPUT DRIVE"
- moved on the sheet: C17, C19, C3, C4, C5, C6, IC4A, IC4B, IC4C, IC4D, IC5A, IC5B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

Commit message: and more
Connections:
- net N$26 renamed TO_ATT1
- net N$35 renamed TO_ATT4
- net N$59 renamed FR_ATT1
- removed net N$29: C4.2, IC4C.OUT, R16.1, TO_ATT2.1
- removed net N$32: C5.2, IC5A.OUT, R19.1, TO_ATT3.1
- new net TO_ATT2: C4.2, IC5A.OUT, R16.1, TO_ATT2.1
- new net TO_ATT3: C5.2, IC4C.OUT, R19.1, TO_ATT3.1
- net N$31: now also SIGOUT3.1; no longer SIGOUT2.1
- net N$34: now also SIGOUT2.1; no longer SIGOUT3.1
- net VCAOUT2: now also IC5A.+IN; no longer IC4C.+IN
- net VCAOUT3: now also IC4C.+IN; no longer IC5A.+IN
Other:
- note removed: "PWM FILTERING AND VCA STATUS LED DRIVE"
- moved on the sheet: +5V, AGND1, AGND2, AGND3, AGND4, C1, C10, C11, C12, C13, C14, C15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

Commit message: MORE
Parts:
- removed C25: (no value), rcl:CPOL-EUE2.5-7
- removed OK1: 6N138, optocoupler:6N138
- removed U$1: 0805DIODE, jasons_stuff:0805DIODE
- added D14: (no value), diode:DIODE-SOD123
- added F1, F2: (no value), adafruit:PTCFUSE-1206
- added IC7: TL074D, linear:TL074D
- added L1, L2: (no value), wuerth-elektronik:WE-CBF_0805
- added R60: (no value), rcl:R-EU_R0805
- C20: device rcl:CPOL-EUE2.5-5 -> rcl:C-EUC0805
- C22, C23: device rcl:C-EUC0805 -> rcl:CPOL-EUE2.5-7
- C24: device rcl:CPOL-EUE2.5-7 -> rcl:CPOL-EUE2.5-5
- D11: value (none) -> 0805DIODE; device microbuilder:DIODESOD-123 -> jasons_stuff:0805DIODE
- D12: value 1N4004 -> (none); device jasons_stuff:1N4004 -> microbuilder:DIODESOD-123
- D13: value 1N4004 -> (none); device jasons_stuff:1N4004 -> diode:DIODE-SOD123
- IC1: value PIC16F1829SOIC -> 74HC595D; device jason_eagle6:PIC16F1829SOIC -> 74xx-eu:74HC595D
- IC2: value V2164 -> TL074D; device jason_eagle6:V2164 -> linear:TL074D
- IC3: value 74HC595D -> PIC16F1829SOIC; device 74xx-eu:74HC595D -> jason_eagle6:PIC16F1829SOIC
- IC6: value TL074D -> V2164; device linear:TL074D -> jason_eagle6:V2164
- IC8: value TL074D -> REG1117; device linear:TL074D -> burr-brown:REG1117
- IC9: value REG1117 -> 6N138; device burr-brown:REG1117 -> optocoupler:6N138
- R25: device rcl:R-EU_R0805 -> rcl:C-EUC0805
- renumbered T1 to Q3, T2 to Q2, T3 to Q1, T4 to Q4
Connections:
- new net N$32: D13.C, F1.1, L1.2
- new net N$35: D14.A, F2.1, L2.2
- net +12V: now also C15.1, C22.+, C3.2, C6.2, C7.1, IC6.V+, IC7P.V+, IC8.VIN, L1.1, R46.2; no longer C17.1, C2.1, C21.2, C22.2, C24.+, D12.A, IC2.V+, IC8P.V+, IC9.VIN, R33.2
- net +5V: now also C2.2, C24.+, C4.2, D10.C, D6.C, D7.C, D8.C, D9.C, IC1A.SCL, IC1P.VCC, IC2P.V+, IC3.VDD, IC8.VOUT, IC9.VCC, R25.2, R28.2; no longer C14.2, C16.2, C20.+, C23.2, D11.C, D2.C, D3.C, D4.C, D5.C, IC1.VDD, IC3A.SCL, IC3P.VCC, IC6P.V+, IC9.VOUT, OK1.VCC, R48.2
- net -12V: now also C23.-, C6.1, C7.2, D12.A, IC6.V-, IC7P.V-, L2.1; no longer C11.1, C17.2, C25.-, D1.A, D13.C, IC2.V-, IC8P.V-
- net AGND: now also C11.1, C14.1, C15.2, C16.1, C17.1, C21.2, C22.-, C23.+, D12.C, D13.A, D14.C, IC6.GND, IC7A.-IN, IC7B.-IN, IC7C.-IN, IC7D.-IN, R31.1, R38.2, R41.2; no longer C10.1, C11.2, C15.1, C18.1, C2.2, C24.-, C25.+, C7.1, D1.C, IC2.GND, IC5A.-IN, IC5B.-IN, IC5C.-IN, IC5D.-IN, R35.2, R39.2, R54.1
- net CKIN: now also D1.A, D6.A, IC3.RA0, R14.2, R5.2; no longer D10.A, D11.A, IC1.RA0, R53.2, R59.2
- net EN_SRC1: now also IC3.RB7, R3.2; no longer IC1.RB7, R9.2
- net EN_SRC2: now also IC3.RC7, R2.2; no longer IC1.RC7, R10.2
- net EN_SRC3: now also IC3.RC4, R1.2; no longer IC1.RC4, R11.2
- net EN_SRC4: now also IC1A.SER, IC3.RB6, R4.2; no longer IC1.RB6, IC3A.SER, R12.2
- net FR_ATT1: now also R56.2; no longer R14.2
- net GATE1: now also D7.A, IC3.RB4, R13.2, R6.2; no longer D6.A, IC1.RB4, R49.2, R55.2
- net GATE2: now also D8.A, IC3.RC2, R12.2, R7.2; no longer D7.A, IC1.RC2, R50.2, R56.2
- net GATE3: now also D9.A, IC3.RC1, R11.2, R8.2; no longer D8.A, IC1.RC1, R51.2, R57.2
- net GATE4: now also D10.A, IC3.RC0, R10.2, R9.2; no longer D9.A, IC1.RC0, R52.2, R58.2
- net GND: now also C2.1, C24.-, C3.1, C4.1, D1.C, D2.C, D3.C, D4.C, D5.C, IC1A.G, IC1P.GND, IC2P.V-, IC3.VSS, IC8.GND, R25.1, R30.2, R31.2, R5.1, R6.1, R7.1, R8.1, R9.1; no longer C14.1, C16.1, C20.-, C22.1, C23.1, D10.C, D6.C, D7.C, D8.C, D9.C, IC1.VSS, IC3A.G, IC3P.GND, IC6P.V-, OK1.GND, R47.2, R54.2, R55.1, R56.1, R57.1, R58.1, R59.1
- net KB_READ: now also IC3.RA1; no longer IC1.RA1
- net MIDI_RX: now also IC3.RB5, IC9.VO, R28.1; no longer IC1.RB5, OK1.VO, R48.1
- net N$1: now also IC1A.QH, R22.2; no longer IC3A.QH, R1.2
- net N$10: now also R21.1; no longer R2.1
- net N$11: now also R20.1; no longer R3.1
- net N$12: now also R19.1; no longer R4.1
- net N$13: now also R18.1; no longer R5.1
- net N$14: now also R17.1; no longer R6.1
- net N$15: now also R16.1; no longer R7.1
- net N$16: now also R15.1; no longer R8.1
- net N$2: now also IC1A.QG, R21.2; no longer IC3A.QG, R2.2
- net N$21: now also IC6.MODE, R46.1; no longer IC2.MODE, R33.1
- net N$22: now also R3.1; no longer R9.1
- net N$23: now also R2.1; no longer R10.1
- net N$24: now also R1.1; no longer R11.1
- net N$25: now also R4.1; no longer R12.1
- net N$27: now also IC7B.+IN, R56.1, R57.2; no longer IC4B.+IN, R14.1, R15.2
- net N$28: now also IC7B.OUT, R57.1; no longer IC4B.OUT, R15.1
- net N$3: now also IC1A.QF, R20.2; no longer IC3A.QF, R3.2
- net N$30: now also IC7D.+IN, R58.2, R59.1; no longer IC4D.+IN, R17.1, R18.2
- net N$31: now also IC7D.OUT, R58.1; no longer IC4D.OUT, R18.1
- net N$33: now also IC4B.+IN, R33.1, R34.2; no longer IC5B.+IN, R20.1, R21.2
- net N$34: now also IC4B.OUT, R34.1; no longer IC5B.OUT, R21.1
- net N$36: now also IC4D.+IN, R35.2, R36.1; no longer IC5D.+IN, R23.1, R24.2
- net N$37: now also IC4D.OUT, R35.1; no longer IC5D.OUT, R24.1
- net N$38: now also C13.2, R47.2; no longer C7.2, R26.2
- net N$39: now also R48.2; no longer R25.2
- net N$4: now also IC1A.QE, R19.2; no longer IC3A.QE, R4.2
- net N$40: now also C14.2, R50.2; no longer C8.2, R28.2
- net N$41: now also R49.2; no longer R27.2
- net N$42: now also C17.2, R54.2; no longer C9.2, R30.2
- net N$43: now also R53.2; no longer R29.2
- net N$44: now also C16.2, R51.2; no longer C10.2, R32.2
- net N$45: now also R52.2; no longer R31.2
- net N$46: now also R24.1; no longer R34.1
- net N$47: now also IC2A.-IN, IC2A.OUT, R24.2; no longer IC6A.-IN, IC6A.OUT, R34.2
- net N$48: now also C8.2, IC5A.+IN, R38.1, R39.2; no longer C12.2, IC8A.+IN, R35.1, R38.2
- net N$5: now also IC1A.QD, R18.2; no longer IC3A.QD, R5.2
- net N$50: now also IC2B.-IN, IC2B.OUT, R27.2; no longer IC6B.-IN, IC6B.OUT, R36.2
- net N$51: now also R27.1; no longer R36.1
- net N$52: now also C9.2, IC5B.+IN, R40.2, R41.1; no longer C13.2, IC8B.+IN, R37.2, R39.1
- net N$53: now also IC2C.-IN, IC2C.OUT, R26.2; no longer IC6C.-IN, IC6C.OUT, R40.2
- net N$54: now also R26.1; no longer R40.1
- net N$55: now also C12.2, IC5C.+IN, R44.2, R45.1; no longer C15.2, IC8C.+IN, R41.2, R42.1
- net N$56: now also IC2D.-IN, IC2D.OUT, R23.2; no longer IC6D.-IN, IC6D.OUT, R43.2
- net N$57: now also R23.1; no longer R43.1
- net N$58: now also C11.2, IC5D.+IN, R42.1, R43.2; no longer C18.2, IC8D.+IN, R44.2, R45.1
- net N$6: now also IC1A.QC, R17.2; no longer IC3A.QC, R6.2
- net N$60: now also R33.2; no longer R20.2
- net N$61: now also R13.1; no longer R49.1
- net N$62: now also IC9.VB, R30.1; no longer OK1.VB, R47.1
- net N$63: now also F2.2; no longer D13.A
- net N$64: now also D11.P$2, IC9.A, R29.2; no longer OK1.A, R46.2, U$1.P$2
- net N$65: now also D11.P$1, IC9.C; no longer OK1.C, U$1.P$1
- net N$66: now also R29.1; no longer R46.1
- net N$67: now also R12.1; no longer R50.1
- net N$68: now also R11.1; no longer R51.1
- net N$69: now also R10.1; no longer R52.1
- net N$7: now also IC1A.QB, R16.2; no longer IC3A.QB, R7.2
- net N$70: now also R59.2; no longer R17.2
- net N$71: now also R36.2; no longer R23.2
- net N$74: now also R14.1; no longer R53.1
- net N$75: now also F1.2; no longer D12.C
- net N$8: now also IC1A.QA, R15.2; no longer IC3A.QA, R8.2
- net N$9: now also R22.1; no longer R1.1
- net PWM1: now also IC2A.+IN, IC3.RC3, R39.1; no longer IC1.RC3, IC6A.+IN, R38.1
- net PWM2: now also IC2B.+IN, IC3.RC6, R40.1; no longer IC1.RC6, IC6B.+IN, R37.1
- net PWM3: now also IC2C.+IN, IC3.RA2, R44.1; no longer IC1.RA2, IC6C.+IN, R41.1
- net PWM4: now also IC2D.+IN, IC3.RC5, R43.1; no longer IC1.RC5, IC6D.+IN, R44.1
- net SR_RCK: now also IC1A.RCK, IC3.RA5; no longer IC1.RA5, IC3A.RCK
- net SR_SCK: now also IC1A.SCK, IC3.RA4; no longer IC1.RA4, IC3A.SCK
- net SWITCH: now also IC3.RA3/MC#; no longer IC1.RA3/MC#
- net TO_ATT1: now also C18.2, IC7A.OUT, R55.1; no longer C3.2, IC4A.OUT, R13.1
- net TO_ATT2: now also C5.2, IC4A.OUT, R32.1; no longer C4.2, IC5A.OUT, R16.1
- net TO_ATT3: now also C20.2, IC7C.OUT, R60.1; no longer C5.2, IC4C.OUT, R19.1
- net TO_ATT4: now also C10.2, IC4C.OUT, R37.1; no longer C6.2, IC5C.OUT, R22.1
- net VCACV1: now also IC5A.-IN, IC5A.OUT, IC6.CVA; no longer IC2.CVA, IC8A.-IN, IC8A.OUT
- net VCACV2: now also IC5B.-IN, IC5B.OUT, IC6.CVB; no longer IC2.CVB, IC8B.-IN, IC8B.OUT
- net VCACV3: now also IC5C.-IN, IC5C.OUT, IC6.CVC; no longer IC2.CVC, IC8C.-IN, IC8C.OUT
- net VCACV4: now also IC5D.-IN, IC5D.OUT, IC6.CVD; no longer IC2.CVD, IC8D.-IN, IC8D.OUT
- net VCAIN1: now also IC6.INA, R47.1, R48.1; no longer IC2.INA, R25.1, R26.1
- net VCAIN2: now also IC6.INB, R49.1, R50.1; no longer IC2.INB, R27.1, R28.1
- net VCAIN3: now also IC6.INC, R53.1, R54.1; no longer IC2.INC, R29.1, R30.1
- net VCAIN4: now also IC6.IND, R51.1, R52.1; no longer IC2.IND, R31.1, R32.1
- net VCAOUT1: now also C18.1, IC6.OUTA, IC7A.+IN, R55.2; no longer C3.1, IC2.OUTA, IC4A.+IN, R13.2
- net VCAOUT2: now also C5.1, IC4A.+IN, IC6.OUTB, R32.2; no longer C4.1, IC2.OUTB, IC5A.+IN, R16.2
- net VCAOUT3: now also C20.1, IC6.OUTC, IC7C.+IN, R60.2; no longer C5.1, IC2.OUTC, IC4C.+IN, R19.2
- net VCAOUT4: now also C10.1, IC4C.+IN, IC6.OUTD, R37.2; no longer C6.1, IC2.OUTD, IC5C.+IN, R22.2
Other:
- moved on the sheet: C10, C11, C12, C13, C14, C15, C16, C17, C18, C2, C21, C24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

Commit message: more
Parts:
- removed AGND1, AGND3: (no value), pinhead:PINHD-1X1
- removed D13, D14: (no value), diode:DIODE-SOD123
- added +12V, -12V: (no value), pinhead:PINHD-1X1
- added C25, C26, C27: (no value), rcl:C-EUC0805
- added D15, D16: 1N4004, jasons_stuff:1N4004
- F1, F2: device adafruit:PTCFUSE-1206 -> microbuilder:PTC1210
- renumbered J1 to ICSP, JP1 to POWER
Connections:
- net +12V: now also +12V.1
- net -12V: now also -12V.1, C25.2, C26.2, C27.1; no longer C19.1, C6.1, C7.2
- net AGND: now also C19.1, C25.1, C26.1, C27.2, C6.1, C7.2, D15.A, D16.C; no longer AGND1.1, AGND3.1, D13.A, D14.C
- net N$32: now also D15.C, F1.2; no longer D13.C, F1.1
- net N$35: now also D16.A, F2.2; no longer D14.A, F2.1
- net N$63: now also F2.1; no longer F2.2
- net N$75: now also F1.1; no longer F1.2
Other:
- moved on the sheet: AGND2, C19, C6, L1, L2

Commit message: fixes
Parts:
- added D13, D14, D17, D18, D19, D20, D21, D22: 0805DIODE, jasons_stuff:0805DIODE
Connections:
- new net N$26: D13.P$1, SINK8.1
- new net N$29: D14.P$1, SINK7.1
- new net N$49: D17.P$1, SINK6.1
- new net N$59: D18.P$1, SINK5.1
- new net N$72: D19.P$1, SINK4.1
- new net N$73: D20.P$1, SINK3.1
- new net N$76: D21.P$1, SINK2.1
- new net N$77: D22.P$1, SINK1.1
- net AGND: now also IC4A.+IN, IC4B.+IN, IC4C.+IN, IC4D.+IN, IC7A.+IN, IC7B.+IN, IC7C.+IN, IC7D.+IN; no longer IC4A.-IN, IC4B.-IN, IC4C.-IN, IC4D.-IN, IC7A.-IN, IC7B.-IN, IC7C.-IN, IC7D.-IN
- net CKIN: now also D1.C; no longer D1.A
- net GATE1: now also D2.C; no longer D2.A
- net GATE2: now also D3.C; no longer D3.A
- net GATE3: now also D4.C; no longer D4.A
- net GATE4: now also D5.C; no longer D5.A
- net GND: now also D1.A, D2.A, D3.A, D4.A, D5.A; no longer D1.C, D2.C, D3.C, D4.C, D5.C
- net N$10: now also D14.P$2; no longer SINK7.1
- net N$11: now also D17.P$2; no longer SINK6.1
- net N$12: now also D18.P$2; no longer SINK5.1
- net N$13: now also D19.P$2; no longer SINK4.1
- net N$14: now also D20.P$2; no longer SINK3.1
- net N$15: now also D21.P$2; no longer SINK2.1
- net N$16: now also D22.P$2; no longer SINK1.1
- net N$27: now also IC7B.-IN; no longer IC7B.+IN
- net N$30: now also IC7D.-IN; no longer IC7D.+IN
- net N$33: now also IC4B.-IN; no longer IC4B.+IN
- net N$36: now also IC4D.-IN; no longer IC4D.+IN
- net N$9: now also D13.P$2; no longer SINK8.1
- net VCAOUT1: now also IC7A.-IN; no longer IC7A.+IN
- net VCAOUT2: now also IC4A.-IN; no longer IC4A.+IN
- net VCAOUT3: now also IC7C.-IN; no longer IC7C.+IN
- net VCAOUT4: now also IC4C.-IN; no longer IC4C.+IN
Other:
- moved on the sheet: D1, D2, D3, D4, D5, IC4A, IC4B, IC4C, IC4D, IC7A, IC7B, IC7C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

Commit message: fixes
Parts:
- D15, D16: value 1N4004 -> MBR0520LT; device jasons_stuff:1N4004 -> diode:MBR0520LT
Changed lines of the file:
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@@
 <part name="F1" library="microbuilder" deviceset="PTC" device="1210"/>
 <part name="F2" library="microbuilder" deviceset="PTC" device="1210"/>
-<part name="D15" library="jasons_stuff" deviceset="1N4004" device=""/>
-<part name="D16" library="jasons_stuff" deviceset="1N4004" device=""/>
 <part name="L1" library="wuerth-elektronik" deviceset="WE-CBF" device="_0805"/>
 <part name="L2" library="wuerth-elektronik" deviceset="WE-CBF" device="_0805"/>
@@
 <part name="D21" library="jasons_stuff" deviceset="0805DIODE" device=""/>
 <part name="D22" library="jasons_stuff" deviceset="0805DIODE" device=""/>
+<part name="D15" library="diode" deviceset="MBR0520LT" device=""/>
+<part name="D16" library="diode" deviceset="MBR0520LT" device=""/>
 </parts>
 <sheets>
@@
 <instance part="F1" gate="G$1" x="27.94" y="284.48"/>
 <instance part="F2" gate="G$1" x="27.94" y="264.16"/>
-<instance part="D15" gate="1" x="17.78" y="279.4" rot="R90"/>
-<instance part="D16" gate="1" x="17.78" y="269.24" rot="R90"/>
 <instance part="L1" gate="G$1" x="5.08" y="281.94"/>
 <instance part="L2" gate="G$1" x="5.08" y="261.62"/>
@@
 <instance part="D21" gate="G$1" x="22.86" y="109.22"/>
 <instance part="D22" gate="G$1" x="30.48" y="109.22"/>
+<instance part="D15" gate="G$1" x="17.78" y="279.4" smashed="yes" rot="R90">
+<attribute name="NAME" x="17.2974" y="281.94" size="1.778" layer="95" rot="R90"/>
+</instance>
+<instance part="D16" gate="G$1" x="17.78" y="269.24" smashed="yes" rot="R90">
+<attribute name="NAME" x="17.2974" y="271.78" size="1.778" layer="95" rot="R90"/>
+</instance>
 </instances>
 <busses>
@@
 <wire x1="-15.24" y1="276.86" x2="-15.24" y2="274.32" width="0.1524" layer="91"/>
 <wire x1="-15.24" y1="274.32" x2="-15.24" y2="271.78" width="0.1524" layer="91"/>
-<wire x1="40.64" y1="274.32" x2="17.78" y2="274.32" width="0.1524" layer="91"/>
 <junction x="-15.24" y="274.32"/>
 <pinref part="SUPPLY35" gate="G$1" pin="AGND"/>
+<wire x1="40.64" y1="274.32" x2="17.78" y2="274.32" width="0.1524" layer="91"/>
 <wire x1="17.78" y1="274.32" x2="-15.24" y2="274.32" width="0.1524" layer="91"/>
 <wire x1="-15.24" y1="274.32" x2="-20.32" y2="274.32" width="0.1524" layer="91"/>
 <wire x1="-20.32" y1="274.32" x2="-20.32" y2="271.78" width="0.1524" layer="91"/>
-<pinref part="D15" gate="1" pin="A"/>
-<wire x1="17.78" y1="276.86" x2="17.78" y2="274.32" width="0.1524" layer="91"/>
+<pinref part="D16" gate="G$1" pin="C"/>
+<wire x1="17.78" y1="271.78" x2="17.78" y2="274.32" width="0.1524" layer="91"/>
 <junction x="17.78" y="274.32"/>
-<pinref part="D16" gate="1" pin="C"/>
-<wire x1="17.78" y1="274.32" x2="17.78" y2="271.78" width="0.1524" layer="91"/>
+<pinref part="D15" gate="G$1" pin="A"/>
+<wire x1="17.78" y1="274.32" x2="17.78" y2="276.86" width="0.1524" layer="91"/>
 </segment>
 <segment>
@@
 <segment>
 <pinref part="F1" gate="G$1" pin="2"/>
-<pinref part="D15" gate="1" pin="C"/>
+<wire x1="10.16" y1="284.48" x2="17.78" y2="284.48" width="0.1524" layer="91"/>
+<pinref part="L1" gate="G$1" pin="2"/>
+<pinref part="D15" gate="G$1" pin="C"/>
 <wire x1="17.78" y1="284.48" x2="22.86" y2="284.48" width="0.1524" layer="91"/>
 <wire x1="17.78" y1="281.94" x2="17.78" y2="284.48" width="0.1524" layer="91"/>
 <junction x="17.78" y="284.48"/>
-<wire x1="10.16" y1="284.48" x2="17.78" y2="284.48" width="0.1524" layer="91"/>
-<pinref part="L1" gate="G$1" pin="2"/>
 </segment>
 </net>
@@
 <segment>
 <pinref part="F2" gate="G$1" pin="2"/>
-<pinref part="D16" gate="1" pin="A"/>
+<wire x1="10.16" y1="264.16" x2="17.78" y2="264.16" width="0.1524" layer="91"/>
+<pinref part="L2" gate="G$1" pin="2"/>
+<pinref part="D16" gate="G$1" pin="A"/>
 <wire x1="17.78" y1="264.16" x2="22.86" y2="264.16" width="0.1524" layer="91"/>
 <wire x1="17.78" y1="266.7" x2="17.78" y2="264.16" width="0.1524" layer="91"/>
 <junction x="17.78" y="264.16"/>
-<wire x1="10.16" y1="264.16" x2="17.78" y2="264.16" width="0.1524" layer="91"/>
-<pinref part="L2" gate="G$1" pin="2"/>
-</segment>
-</net>
+</segment>
+</net>
