File: main_board/main_board.sch (EAGLE design)
At the start: 176 parts, among them IC1 74HC595D, IC2 TL074D, IC3 PIC16F1829SOIC, IC4 TL074D, IC5 TL074D, IC6 V2164, IC7 TL074D, IC8 REG1117, IC9 6N138

Commit message: fixes
Parts:
- removed CLOCKIN: (no value), pinhead:PINHD-1X1
- removed D1, D6: (no value), microbuilder:DIODESOD-123
- removed R14, R5: (no value), rcl:R-EU_R0805
- added GND1: (no value), pinhead:PINHD-1X1
Connections:
- removed net N$74: CLOCKIN.1, R14.1
- net +5V: no longer D6.C
- net CKIN: no longer D1.C, D6.A, R14.2, R5.2
- net GND: now also GND1.1; no longer D1.A, R5.1
Changed lines of the file:
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@@
 <part name="SUPPLY30" library="supply2" deviceset="+5V" device=""/>
 <part name="GND15" library="supply1" deviceset="GND" device=""/>
-<part name="CLOCKIN" library="pinhead" deviceset="PINHD-1X1" device=""/>
-<part name="R14" library="rcl" deviceset="R-EU_" device="R0805"/>
-<part name="D1" library="microbuilder" deviceset="DIODE" device="SOD-123"/>
-<part name="D6" library="microbuilder" deviceset="DIODE" device="SOD-123"/>
 <part name="SWITCH" library="pinhead" deviceset="PINHD-1X1" device=""/>
 <part name="IC8" library="burr-brown" deviceset="REG1117" device=""/>
@@
 <part name="R8" library="rcl" deviceset="R-EU_" device="R0805"/>
 <part name="R9" library="rcl" deviceset="R-EU_" device="R0805"/>
-<part name="R5" library="rcl" deviceset="R-EU_" device="R0805"/>
 <part name="GND16" library="supply1" deviceset="GND" device=""/>
 <part name="C19" library="rcl" deviceset="C-EU" device="C0805"/>
@@
 <part name="D15" library="diode" deviceset="MBR0520LT" device=""/>
 <part name="D16" library="diode" deviceset="MBR0520LT" device=""/>
+<part name="GND1" library="pinhead" deviceset="PINHD-1X1" device=""/>
 </parts>
 <sheets>
@@
 <instance part="SUPPLY30" gate="+5V" x="-93.98" y="76.2"/>
 <instance part="GND15" gate="1" x="-114.3" y="2.54"/>
-<instance part="CLOCKIN" gate="G$1" x="-137.16" y="27.94" rot="R180"/>
-<instance part="R14" gate="G$1" x="-121.92" y="27.94"/>
-<instance part="D1" gate="G$1" x="-109.22" y="25.4"/>
-<instance part="D6" gate="G$1" x="-99.06" y="30.48"/>
 <instance part="SWITCH" gate="G$1" x="58.42" y="20.32" rot="R270"/>
 <instance part="IC8" gate="G$1" x="-91.44" y="279.4"/>
@@
 <instance part="GND21" gate="G$1" x="48.26" y="152.4" rot="R180"/>
 <instance part="GND22" gate="G$1" x="48.26" y="142.24" rot="R180"/>
-<instance part="GND25" gate="1" x="58.42" y="132.08"/>
+<instance part="GND25" gate="1" x="58.42" y="119.38"/>
 <instance part="+5V" gate="G$1" x="48.26" y="162.56" rot="R180"/>
 <instance part="SUPPLY41" gate="+5V" x="58.42" y="167.64"/>
@@
 <instance part="R8" gate="G$1" x="-81.28" y="17.78" rot="R90"/>
 <instance part="R9" gate="G$1" x="-78.74" y="17.78" rot="R90"/>
-<instance part="R5" gate="G$1" x="-76.2" y="17.78" rot="R90"/>
 <instance part="GND16" gate="1" x="-86.36" y="2.54"/>
 <instance part="C19" gate="G$1" x="96.52" y="167.64" rot="R180"/>
@@
 <attribute name="NAME" x="17.2974" y="271.78" size="1.778" layer="95" rot="R90"/>
 </instance>
+<instance part="GND1" gate="G$1" x="48.26" y="132.08" rot="R180"/>
 </instances>
 <busses>
@@
 <wire x1="-93.98" y1="73.66" x2="-93.98" y2="71.12" width="0.1524" layer="91"/>
 <junction x="-93.98" y="71.12"/>
-<pinref part="D6" gate="G$1" pin="C"/>
-<wire x1="-96.52" y1="30.48" x2="-93.98" y2="30.48" width="0.1524" layer="91"/>
-<wire x1="-93.98" y1="30.48" x2="-93.98" y2="40.64" width="0.1524" layer="91"/>
-<junction x="-93.98" y="40.64"/>
 </segment>
 <segment>
@@
 </segment>
 <segment>
-<wire x1="-114.3" y1="5.08" x2="-114.3" y2="25.4" width="0.1524" layer="91"/>
+<wire x1="-114.3" y1="5.08" x2="-114.3" y2="35.56" width="0.1524" layer="91"/>
 <pinref part="GND15" gate="1" pin="GND"/>
 <pinref part="D2" gate="G$1" pin="A"/>
-<wire x1="-114.3" y1="25.4" x2="-114.3" y2="35.56" width="0.1524" layer="91"/>
 <wire x1="-114.3" y1="35.56" x2="-114.3" y2="45.72" width="0.1524" layer="91"/>
 <wire x1="-114.3" y1="45.72" x2="-114.3" y2="55.88" width="0.1524" layer="91"/>
@@
 <wire x1="-111.76" y1="35.56" x2="-114.3" y2="35.56" width="0.1524" layer="91"/>
 <junction x="-114.3" y="35.56"/>
-<pinref part="D1" gate="G$1" pin="A"/>
-<wire x1="-111.76" y1="25.4" x2="-114.3" y2="25.4" width="0.1524" layer="91"/>
-<junction x="-114.3" y="25.4"/>
 </segment>
 <segment>
@@
 <wire x1="58.42" y1="152.4" x2="58.42" y2="142.24" width="0.1524" layer="91"/>
 <pinref part="GND22" gate="G$1" pin="1"/>
-<wire x1="58.42" y1="142.24" x2="58.42" y2="134.62" width="0.1524" layer="91"/>
+<wire x1="58.42" y1="142.24" x2="58.42" y2="132.08" width="0.1524" layer="91"/>
+<wire x1="58.42" y1="132.08" x2="58.42" y2="121.92" width="0.1524" layer="91"/>
 <wire x1="50.8" y1="142.24" x2="58.42" y2="142.24" width="0.1524" layer="91"/>
 <junction x="58.42" y="142.24"/>
 <pinref part="GND25" gate="1" pin="GND"/>
+<pinref part="GND1" gate="G$1" pin="1"/>
+<wire x1="50.8" y1="132.08" x2="58.42" y2="132.08" width="0.1524" layer="91"/>
+<junction x="58.42" y="132.08"/>
 </segment>
 <segment>
@@
 <wire x1="-78.74" y1="10.16" x2="-78.74" y2="12.7" width="0.1524" layer="91"/>
 <junction x="-81.28" y="10.16"/>
-<pinref part="R5" gate="G$1" pin="1"/>
-<wire x1="-78.74" y1="10.16" x2="-76.2" y2="10.16" width="0.1524" layer="91"/>
-<wire x1="-76.2" y1="10.16" x2="-76.2" y2="12.7" width="0.1524" layer="91"/>
-<junction x="-78.74" y="10.16"/>
 </segment>
 </net>
@@
 <pinref part="R10" gate="G$1" pin="1"/>
 <wire x1="-134.62" y1="38.1" x2="-127" y2="38.1" width="0.1524" layer="91"/>
-</segment>
-</net>
-<net name="N$74" class="0">
-<segment>
-<pinref part="CLOCKIN" gate="G$1" pin="1"/>
-<pinref part="R14" gate="G$1" pin="1"/>
-<wire x1="-134.62" y1="27.94" x2="-127" y2="27.94" width="0.1524" layer="91"/>
 </segment>
 </net>
@@
 <net name="CKIN" class="0">
 <segment>
-<pinref part="R14" gate="G$1" pin="2"/>
-<wire x1="-116.84" y1="27.94" x2="-104.14" y2="27.94" width="0.1524" layer="91"/>
-<wire x1="-104.14" y1="25.4" x2="-104.14" y2="27.94" width="0.1524" layer="91"/>
-<junction x="-104.14" y="27.94"/>
-<wire x1="-104.14" y1="27.94" x2="-104.14" y2="30.48" width="0.1524" layer="91"/>
-<pinref part="D6" gate="G$1" pin="A"/>
-<wire x1="-104.14" y1="30.48" x2="-101.6" y2="30.48" width="0.1524" layer="91"/>
-<label x="-66.04" y="27.94" size="1.778" layer="95"/>
-<wire x1="-104.14" y1="27.94" x2="-76.2" y2="27.94" width="0.1524" layer="91"/>
-<pinref part="R5" gate="G$1" pin="2"/>
-<wire x1="-76.2" y1="27.94" x2="-60.96" y2="27.94" width="0.1524" layer="91"/>
-<wire x1="-76.2" y1="22.86" x2="-76.2" y2="27.94" width="0.1524" layer="91"/>
-<junction x="-76.2" y="27.94"/>
-<pinref part="D1" gate="G$1" pin="C"/>
-<wire x1="-106.68" y1="25.4" x2="-104.14" y2="25.4" width="0.1524" layer="91"/>
-</segment>
-<segment>
 <pinref part="IC3" gate="G$1" pin="RA0"/>
